File: Module_PCB/LEDStripModule.sch (KiCad schematic (older format))
At the start: 107 parts, among them J2 ISP, J4 DS, J5 US, Q1 KIA50N03B, Q2 KIA50N03B, Q3 KIA50N03B, Q4 KIA50N03B, U1 W25Q16JV, U2 AP1117-33, U3 TPS563200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

Commit message: Fixed pin header part numbers
Parts:
- J4: MPN SQT-102-01-F-D-RA -> A2541HWR-2x2P; Manufacturer Samtec -> CJT(Changjiang Connectors)
- J5: MPN TMM-102-01-T-D-RA -> PZ254R-12-4P; Manufacturer Samtec -> XFCN
Changed lines of the file:
@@
 F 2 "Connector_PinSocket_2.54mm:PinSocket_2x02_P2.54mm_Horizontal" H 5650 5650 50  0001 C CNN
 F 3 "~" H 5650 5650 50  0001 C CNN
-F 4 "Samtec" H 5650 5650 50  0001 C CNN "Manufacturer"
-F 5 "SQT-102-01-F-D-RA" H 5650 5650 50  0001 C CNN "MPN"
+F 4 "CJT(Changjiang Connectors)" H 5650 5650 50  0001 C CNN "Manufacturer"
+F 5 "A2541HWR-2x2P" H 5650 5650 50  0001 C CNN "MPN"
 	1    5650 5650
 	1    0    0    -1
@@
 F 2 "Connector_PinHeader_2.54mm:PinHeader_2x02_P2.54mm_Horizontal" H 5650 5100 50  0001 C CNN
 F 3 "~" H 5650 5100 50  0001 C CNN
-F 4 "Samtec" H 5650 5100 50  0001 C CNN "Manufacturer"
-F 5 "TMM-102-01-T-D-RA" H 5650 5100 50  0001 C CNN "MPN"
+F 4 "XFCN" H 5650 5100 50  0001 C CNN "Manufacturer"
+F 5 "PZ254R-12-4P" H 5650 5100 50  0001 C CNN "MPN"
 	1    5650 5100
 	1    0    0    -1

Commit message: Added test pads
Parts:
- added TP1: TP, TestPoint:TestPoint_Pad_D2.0mm, symbol Connector:TestPoint
- added TP2: GND, TestPoint:TestPoint_Pad_D2.0mm, symbol Connector:TestPoint
Connections:
- net GND: now also TP2.1
- net LED: now also U5.25 (PC2); no longer U5.23 (PC0)
- net TP1: now reaches U5.24 (PC1)
- net TP1: now also TP1.1
Changed lines of the file:
@@
 	1    0    0    -1
 $EndComp
-Text Label 3200 5600 0    50   ~ 0
+Text Label 3200 5800 0    50   ~ 0
 LED
 $Comp
@@
 $EndComp
 NoConn ~ 7150 5950
+$Comp
+L Connector:TestPoint TP1
+U 1 1 60DA3249
+P 4600 5800
+F 0 "TP1" H 4658 5918 50  0000 L CNN
+F 1 "TP" H 4658 5827 50  0000 L CNN
+F 2 "TestPoint:TestPoint_Pad_D2.0mm" H 4800 5800 50  0001 C CNN
+F 3 "~" H 4800 5800 50  0001 C CNN
+	1    4600 5800
+	1    0    0    -1
+$EndComp
+$Comp
+L Connector:TestPoint TP2
+U 1 1 60DA37C3
+P 4900 5800
+F 0 "TP2" H 4958 5918 50  0000 L CNN
+F 1 "GND" H 4958 5827 50  0000 L CNN
+F 2 "TestPoint:TestPoint_Pad_D2.0mm" H 5100 5800 50  0001 C CNN
+F 3 "~" H 5100 5800 50  0001 C CNN
+	1    4900 5800
+	1    0    0    -1
+$EndComp
+$Comp
+L power:GND #PWR0147
+U 1 1 60DA3BA0
+P 4900 5800
+F 0 "#PWR0147" H 4900 5550 50  0001 C CNN
+F 1 "GND" H 4905 5627 50  0000 C CNN
+F 2 "" H 4900 5800 50  0001 C CNN
+F 3 "" H 4900 5800 50  0001 C CNN
+	1    4900 5800
+	1    0    0    -1
+$EndComp
+Text Label 4600 5800 3    50   ~ 0
+TP1
+Text Label 3200 5700 0    50   ~ 0
+TP1
 $EndSCHEMATC

Commit message: Added MPN for isp header Exported BOM
Parts:
- J2: MPN (none) -> MTP125-1106S1; Manufacturer (none) -> MINTRON
- TP1, TP2: footprint TestPoint:TestPoint_Pad_D2.0mm -> TestPoint:TestPoint_Pad_D1.5mm
Changed lines of the file:
@@
 F 2 "Connector_PinHeader_2.54mm:PinHeader_1x06_P2.54mm_Vertical" H 4200 6000 50  0001 C CNN
 F 3 "~" H 4200 6000 50  0001 C CNN
+F 4 "MINTRON" H 4200 6000 50  0001 C CNN "Manufacturer"
+F 5 "MTP125-1106S1" H 4200 6000 50  0001 C CNN "MPN"
 	1    4200 6000
 	1    0    0    -1
@@
 F 0 "TP1" H 4658 5918 50  0000 L CNN
 F 1 "TP" H 4658 5827 50  0000 L CNN
-F 2 "TestPoint:TestPoint_Pad_D2.0mm" H 4800 5800 50  0001 C CNN
+F 2 "TestPoint:TestPoint_Pad_D1.5mm" H 4800 5800 50  0001 C CNN
 F 3 "~" H 4800 5800 50  0001 C CNN
 	1    4600 5800
@@
 F 0 "TP2" H 4958 5918 50  0000 L CNN
 F 1 "GND" H 4958 5827 50  0000 L CNN
-F 2 "TestPoint:TestPoint_Pad_D2.0mm" H 5100 5800 50  0001 C CNN
+F 2 "TestPoint:TestPoint_Pad_D1.5mm" H 5100 5800 50  0001 C CNN
 F 3 "~" H 5100 5800 50  0001 C CNN
 	1    4900 5800
