File: Module_PCB/Module_PCB.kicad_pcb (KiCad board)
At the start: 2 copper layers, 247.5 x 25 mm, 106 parts, among them J1 ISP, J2 US, J3 DS, Q1 HSS2307, Q2 BSS123, U1 W25Q16JV, U2 AP1117-33, U3 TPS563200, U5 ATmega328P-AU, U7 74LVC1G34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

Commit message: Updated 22u capacitors to 1206 package
Parts:
- C1, C10, C14, C15, C16, C17, C2, C22, C6, C9: footprint Capacitor_SMD:C_0603_1608Metric -> Capacitor_SMD:C_1206_3216Metric
- moved C10 1.43 mm to (66.6, 105.3)
- moved C15 0.99 mm to (193.2, 106.3)
- moved C9 0.83 mm to (66.6, 107.7)
- moved C14 0.70 mm to (264.7, 106.3)
- moved C16 0.70 mm to (149.3, 106.3)
- moved C17 0.70 mm to (22.7, 106.3)
- moved C22 0.70 mm to (88.7, 106.3)
- moved C2 0.56 mm to (170.5, 107.3)
- moved C1 0.40 mm to (67.7, 111.2)
- moved C6 0.36 mm to (172.2, 115.4)
Routing:
- net +4V: track 168.8 -> 170.8 mm
- net GND: track 42.4 -> 41.5 mm
- net +3V3: track 144.7 -> 145.3 mm
