File: main_pcb_adapter/main_pcb_adapter.sch (KiCad schematic (older format))
At the start: 3 parts, among them J1 DN, J2 UP, J3 UPDN

Commit message: Added MPN/MF
Parts:
- J1, J2: MPN (none) -> DS1023-2*3SF11; Manufacturer (none) -> CONNFLY Elec
- J3: MPN (none) -> B-2100S08P-B110; Manufacturer (none) -> Ckmtw(Shenzhen Cankemeng)
Changed lines of the file:
@@
 F 2 "Connector_PinSocket_2.54mm:PinSocket_2x03_P2.54mm_Vertical" H 5450 2750 50  0001 C CNN
 F 3 "~" H 5450 2750 50  0001 C CNN
+F 4 "DS1023-2*3SF11" H 5450 2750 50  0001 C CNN "MPN"
+F 5 "CONNFLY Elec" H 5450 2750 50  0001 C CNN "Manufacturer"
 	1    5450 2750
 	1    0    0    -1
@@
 F 2 "Connector_PinSocket_2.54mm:PinSocket_2x03_P2.54mm_Vertical" H 4000 2750 50  0001 C CNN
 F 3 "~" H 4000 2750 50  0001 C CNN
+F 4 "DS1023-2*3SF11" H 4000 2750 50  0001 C CNN "MPN"
+F 5 "CONNFLY Elec" H 4000 2750 50  0001 C CNN "Manufacturer"
 	1    4000 2750
 	1    0    0    -1
@@
 F 2 "Connector_PinHeader_2.54mm:PinHeader_2x04_P2.54mm_Vertical" H 4650 4050 50  0001 C CNN
 F 3 "~" H 4650 4050 50  0001 C CNN
+F 4 "B-2100S08P-B110" H 4650 4050 50  0001 C CNN "MPN"
+F 5 "Ckmtw(Shenzhen Cankemeng)" H 4650 4050 50  0001 C CNN "Manufacturer"
 	1    4650 4050
 	1    0    0    -1
