File: main_pcb/main_pcb.kicad_pcb (KiCad board)
At the start: 2 copper layers, 95 x 95 mm, 54 parts, among them J1 DBG, J2 UI, J3 UI, J4 Raspberry_Pi_Zero_WH, J5 UI, J6 UI, J7 UPDN, J8 ISP, J9 BTN_TRIG, Q1 BSS123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

Commit message: Moved the LED control from the Pi to the AVR
Parts:
- removed D3: LED, LED_SMD:LED_0603_1608Metric
- removed R19: 330, Resistor_SMD:R_0603_1608Metric
Connections:
- H1 pad 1: Net-(H1-Pad1) -> unconnected-(H1-Pad1)
- H2 pad 1: Net-(H2-Pad1) -> unconnected-(H2-Pad1)
- H3 pad 1: Net-(H3-Pad1) -> unconnected-(H3-Pad1)
- H4 pad 1: Net-(H4-Pad1) -> unconnected-(H4-Pad1)
- J4 pad 11: Net-(J4-Pad11) -> unconnected-(J4-Pad11)
- J4 pad 26: Net-(J4-Pad26) -> unconnected-(J4-Pad26)
- J4 pad 28: Net-(J4-Pad28) -> unconnected-(J4-Pad28)
- J4 pad 29: Net-(J4-Pad29) -> unconnected-(J4-Pad29)
- J4 pad 31: Net-(J4-Pad31) -> unconnected-(J4-Pad31)
- J4 pad 33: /STAT -> unconnected-(J4-Pad33)
- J4 pad 36: Net-(J4-Pad36) -> unconnected-(J4-Pad36)
- J4 pad 37: Net-(J4-Pad37) -> unconnected-(J4-Pad37)
- J5 pad 3: /STAT -> /UC_LED
- J7 pad 7: Net-(J7-Pad7) -> unconnected-(J7-Pad7)
- U1 pad 1: Net-(U1-Pad1) -> unconnected-(U1-Pad1)
- U1 pad 16: Net-(U1-Pad16) -> unconnected-(U1-Pad16)
- U1 pad 17: Net-(U1-Pad17) -> unconnected-(U1-Pad17)
- U1 pad 18: Net-(U1-Pad18) -> unconnected-(U1-Pad18)
- U1 pad 19: Net-(U1-Pad19) -> unconnected-(U1-Pad19)
- U1 pad 2: Net-(U1-Pad2) -> unconnected-(U1-Pad2)
- U1 pad 20: Net-(U1-Pad20) -> unconnected-(U1-Pad20)
- U1 pad 21: Net-(U1-Pad21) -> unconnected-(U1-Pad21)
- U1 pad 25: Net-(U1-Pad25) -> unconnected-(U1-Pad25)
- U1 pad 26: Net-(U1-Pad26) -> unconnected-(U1-Pad26)
- U1 pad 27: Net-(U1-Pad27) -> unconnected-(U1-Pad27)
- U1 pad 28: Net-(U1-Pad28) -> unconnected-(U1-Pad28)
- U3 pad 1: Net-(U3-Pad1) -> unconnected-(U3-Pad1)
- U3 pad 10: Net-(U3-Pad10) -> unconnected-(U3-Pad10)
- U3 pad 11: Net-(U3-Pad11) -> unconnected-(U3-Pad11)
- U3 pad 12: Net-(U3-Pad12) -> unconnected-(U3-Pad12)
- U3 pad 19: Net-(U3-Pad19) -> unconnected-(U3-Pad19)
- U3 pad 2: Net-(U3-Pad2) -> unconnected-(U3-Pad2)
- U3 pad 9: Net-(U3-Pad9) -> unconnected-(U3-Pad9)
Routing:
- net /UC_LED: track 13.2 -> 62.2 mm, vias 0 -> 3
- net /STAT: track 40.2 -> 0.00 mm
- net Net-(D3-Pad2): track 1.69 -> 0.00 mm
- net GND: track 27.0 -> 25.9 mm, vias 24 -> 23
- net /BR+: track 58.4 -> 59.4 mm
- net +3V3: track 205.1 -> 204.6 mm
